File: 10_hw/oceanside_v3/SUB_PERIS.sch (KiCad schematic (older format))
At the start: 23 parts, among them J10 CONSOLECON, J11 SBCUSB, J12 CAN, J13 RS485, U4 FT232R, U5 SN65HVD233-HT, U6 SN65HVD1781A-Q1

Commit message: schematic modified.
CAN IC pin 8 should be connected to GND.
Parts:
- R12: value 10k -> 0
Changed lines of the file:
@@
 P 9350 1850
 F 0 "R12" H 9200 1800 50  0000 C CNN
-F 1 "10k" H 9200 1900 50  0000 C CNN
+F 1 "0" H 9200 1900 50  0000 C CNN
 F 2 "Resistors_SMD:R_0805_HandSoldering" V 9280 1850 50  0001 C CNN
 F 3 "" H 9350 1850 50  0000 C CNN
